Commit message: icub hands with new dh_frames at the center of the hand

File: app/robots/icubGazeboSim/model.urdf (robot description, URDF)
Before this commit: robot iCub, 58 links, 57 joints
Links:
- removed link l_gripper
- removed link r_gripper
- added link l_ai_dummy, mass 0.010
- added link l_ail1, mass 0.010; collision mesh filename=file:///home/yeshi/icub-gazebo/icub/meshes/collision/l_hand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; visual mesh filename=file:///home/yeshi/icub-gazebo/icub/meshes/visual/l_hand/l_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
- added link l_ail2, mass 0.010; collision mesh filename=file:///home/yeshi/icub-gazebo/icub/meshes/collision/l_hand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; visual mesh filename=file:///home/yeshi/icub-gazebo/icub/meshes/visual/l_hand/l_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
- added link l_ail3, mass 0.010; collision mesh filename=file:///home/yeshi/icub-gazebo/icub/meshes/collision/l_hand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; visual mesh filename=file:///home/yeshi/icub-gazebo/icub/meshes/visual/l_hand/l_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
- added link l_li_dummy, mass 0.010
- added link l_lil1, mass 0.010; collision mesh filename=file:///home/yeshi/icub-gazebo/icub/meshes/collision/l_hand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; visual mesh filename=file:///home/yeshi/icub-gazebo/icub/meshes/visual/l_hand/l_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
- added link l_lil2, mass 0.010; collision mesh filename=file:///home/yeshi/icub-gazebo/icub/meshes/collision/l_hand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; visual mesh filename=file:///home/yeshi/icub-gazebo/icub/meshes/visual/l_hand/l_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
- added link l_lil3, mass 0.010; collision mesh filename=file:///home/yeshi/icub-gazebo/icub/meshes/collision/l_hand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; visual mesh filename=file:///home/yeshi/icub-gazebo/icub/meshes/visual/l_hand/l_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
- added link l_ml1, mass 0.010; collision mesh filename=file:///home/yeshi/icub-gazebo/icub/meshes/collision/l_hand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; visual mesh filename=file:///home/yeshi/icub-gazebo/icub/meshes/visual/l_hand/l_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
- added link l_ml2, mass 0.010; collision mesh filename=file:///home/yeshi/icub-gazebo/icub/meshes/collision/l_hand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; visual mesh filename=file:///home/yeshi/icub-gazebo/icub/meshes/visual/l_hand/l_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
- added link l_ml3, mass 0.010; collision mesh filename=file:///home/yeshi/icub-gazebo/icub/meshes/collision/l_hand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; visual mesh filename=file:///home/yeshi/icub-gazebo/icub/meshes/visual/l_hand/l_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
- added link l_ml_dummy, mass 0.010
- added link l_ril1, mass 0.010; collision mesh filename=file:///home/yeshi/icub-gazebo/icub/meshes/collision/l_hand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; visual mesh filename=file:///home/yeshi/icub-gazebo/icub/meshes/visual/l_hand/l_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
- added link l_ril2, mass 0.010; collision mesh filename=file:///home/yeshi/icub-gazebo/icub/meshes/collision/l_hand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; visual mesh filename=file:///home/yeshi/icub-gazebo/icub/meshes/visual/l_hand/l_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
- added link l_ril3, mass 0.010; collision mesh filename=file:///home/yeshi/icub-gazebo/icub/meshes/collision/l_hand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; visual mesh filename=file:///home/yeshi/icub-gazebo/icub/meshes/visual/l_hand/l_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
- added link l_ril_dummy, mass 0.010
- added link l_tl0, mass 0.010; collision mesh filename=file:///home/yeshi/icub-gazebo/icub/meshes/collision/l_hand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; collision mesh filename=file:///home/yeshi/icub-gazebo/icub/meshes/collision/l_hand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
- added link l_tl2, mass 0.010; collision mesh filename=file:///home/yeshi/icub-gazebo/icub/meshes/collision/l_hand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; visual mesh filename=file:///home/yeshi/icub-gazebo/icub/meshes/visual/l_hand/l_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
- added link l_tl3, mass 0.010; collision mesh filename=file:///home/yeshi/icub-gazebo/icub/meshes/collision/l_hand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; visual mesh filename=file:///home/yeshi/icub-gazebo/icub/meshes/visual/l_hand/l_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
- added link l_tl4, mass 0.010; collision mesh filename=file:///home/yeshi/icub-gazebo/icub/meshes/collision/l_hand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; visual mesh filename=file:///home/yeshi/icub-gazebo/icub/meshes/visual/l_hand/l_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
- added link r_ai_dummy, mass 0.010
- added link r_ail1, mass 0.010; collision mesh filename=file:///home/yeshi/icub-gazebo/icub/meshes/collision/r_hand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; visual mesh filename=file:///home/yeshi/icub-gazebo/icub/meshes/visual/r_hand/r_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
- added link r_ail2, mass 0.010; collision mesh filename=file:///home/yeshi/icub-gazebo/icub/meshes/collision/r_hand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; visual mesh filename=file:///home/yeshi/icub-gazebo/icub/meshes/visual/r_hand/r_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
- added link r_ail3, mass 0.010; collision mesh filename=file:///home/yeshi/icub-gazebo/icub/meshes/collision/r_hand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; visual mesh filename=file:///home/yeshi/icub-gazebo/icub/meshes/visual/r_hand/r_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
- added link r_li_dummy, mass 0.010
- added link r_lil1, mass 0.010; collision mesh filename=file:///home/yeshi/icub-gazebo/icub/meshes/collision/r_hand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; visual mesh filename=file:///home/yeshi/icub-gazebo/icub/meshes/visual/r_hand/r_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
- added link r_lil2, mass 0.010; collision mesh filename=file:///home/yeshi/icub-gazebo/icub/meshes/collision/r_hand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; visual mesh filename=file:///home/yeshi/icub-gazebo/icub/meshes/visual/r_hand/r_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
- added link r_lil3, mass 0.010; collision mesh filename=file:///home/yeshi/icub-gazebo/icub/meshes/collision/r_hand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; visual mesh filename=file:///home/yeshi/icub-gazebo/icub/meshes/visual/r_hand/r_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
- added link r_m_dummy, mass 0.010
- added link r_ml1, mass 0.010; collision mesh filename=file:///home/yeshi/icub-gazebo/icub/meshes/collision/r_hand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; visual mesh filename=file:///home/yeshi/icub-gazebo/icub/meshes/visual/r_hand/r_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
- added link r_ml2, mass 0.010; collision mesh filename=file:///home/yeshi/icub-gazebo/icub/meshes/collision/r_hand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; visual mesh filename=file:///home/yeshi/icub-gazebo/icub/meshes/visual/r_hand/r_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
- added link r_ml3, mass 0.010; collision mesh filename=file:///home/yeshi/icub-gazebo/icub/meshes/collision/r_hand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; visual mesh filename=file:///home/yeshi/icub-gazebo/icub/meshes/visual/r_hand/r_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
- added link r_ril1, mass 0.010; collision mesh filename=file:///home/yeshi/icub-gazebo/icub/meshes/collision/r_hand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; visual mesh filename=file:///home/yeshi/icub-gazebo/icub/meshes/visual/r_hand/r_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
- added link r_ril2, mass 0.010; collision mesh filename=file:///home/yeshi/icub-gazebo/icub/meshes/collision/r_hand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; visual mesh filename=file:///home/yeshi/icub-gazebo/icub/meshes/visual/r_hand/r_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
- added link r_ril3, mass 0.010; collision mesh filename=file:///home/yeshi/icub-gazebo/icub/meshes/collision/r_hand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; visual mesh filename=file:///home/yeshi/icub-gazebo/icub/meshes/visual/r_hand/r_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
- added link r_rir_dummy, mass 0.010
- added link r_tl0, mass 0.010; collision mesh filename=file:///home/yeshi/icub-gazebo/icub/meshes/collision/r_hand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; collision mesh filename=file:///home/yeshi/icub-gazebo/icub/meshes/collision/r_hand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
- added link r_tl2, mass 0.010; collision mesh filename=file:///home/yeshi/icub-gazebo/icub/meshes/collision/r_hand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; visual mesh filename=file:///home/yeshi/icub-gazebo/icub/meshes/visual/r_hand/r_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
- added link r_tl3, mass 0.010; collision mesh filename=file:///home/yeshi/icub-gazebo/icub/meshes/collision/r_hand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; visual mesh filename=file:///home/yeshi/icub-gazebo/icub/meshes/visual/r_hand/r_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
- added link r_tl4, mass 0.010; collision mesh filename=file:///home/yeshi/icub-gazebo/icub/meshes/collision/r_hand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; visual mesh filename=file:///home/yeshi/icub-gazebo/icub/meshes/visual/r_hand/r_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
- link chest: geometry collision mesh filename=file:///home/yeshi/icub-gazebo/icub/meshes/collision/icub_s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 scale=1 1 1; visual mesh filename=file:///home/yeshi/icub-gazebo/icub/meshes/visual/icub_ches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 scale=1 1 1
- link head: geometry collision mesh filename=file:///home/yeshi/icub-gazebo/icub/meshes/collision/icub_s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 scale=1 1 1; visual mesh filename=file:///home/yeshi/icub-gazebo/icub/meshes/visual/icub_head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 scale=1 1 1
- link l_ankle_1: geometry collision mesh filename=file:///home/yeshi/icub-gazebo/icub/meshes/collision/icub_s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 scale=1 1 1; visual mesh filename=file:///home/yeshi/icub-gazebo/icub/meshes/visual/icub_l_an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 scale=1 1 1
- link l_foot: geometry collision mesh filename=file:///home/yeshi/icub-gazebo/icub/meshes/collision/icub_s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 scale=1 1 1; visual mesh filename=file:///home/yeshi/icub-gazebo/icub/meshes/visual/icub_l_fo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 scale=1 1 1
- link l_forearm: geometry collision mesh filename=file:///home/yeshi/icub-gazebo/icub/meshes/collision/icub_s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 scale=1 1 1; visual mesh filename=file:///home/yeshi/icub-gazebo/icub/meshes/visual/icub_l_fo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 scale=1 1 1
- link l_hand: mass 0.213 -> 0.010; geometry collision mesh filename=file:///home/yeshi/icub-gazebo/icub/meshes/collision/l_hand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; collision mesh filename=file:///home/yeshi/icub-gazebo/icub/meshes/collision/l_hand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
- link l_hip_1: geometry collision mesh filename=file:///home/yeshi/icub-gazebo/icub/meshes/collision/icub_s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 scale=1 1 1; visual mesh filename=file:///home/yeshi/icub-gazebo/icub/meshes/visual/icub_l_hi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 scale=1 1 1
- link l_hip_2: geometry collision mesh filename=file:///home/yeshi/icub-gazebo/icub/meshes/collision/icub_s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 scale=1 1 1; visual mesh filename=file:///home/yeshi/icub-gazebo/icub/meshes/visual/icub_l_hi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 scale=1 1 1
- link l_lower_leg: geometry collision mesh filename=file:///home/yeshi/icub-gazebo/icub/meshes/collision/icub_s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 scale=1 1 1; visual mesh filename=file:///home/yeshi/icub-gazebo/icub/meshes/visual/icub_l_sh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 scale=1 1 1
- link l_shoulder_1: geometry collision mesh filename=file:///home/yeshi/icub-gazebo/icub/meshes/collision/icub_s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 scale=1 1 1; visual mesh filename=file:///home/yeshi/icub-gazebo/icub/meshes/visual/icub_l_sh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 scale=1 1 1
- link l_shoulder_2: geometry collision mesh filename=file:///home/yeshi/icub-gazebo/icub/meshes/collision/icub_s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 scale=1 1 1; visual mesh filename=file:///home/yeshi/icub-gazebo/icub/meshes/visual/icub_l_sh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 scale=1 1 1
- link l_upper_arm: geometry collision mesh filename=file:///home/yeshi/icub-gazebo/icub/meshes/collision/icub_s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 scale=1 1 1; visual mesh filename=file:///home/yeshi/icub-gazebo/icub/meshes/visual/icub_l_ar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 scale=1 1 1
- link l_upper_leg: geometry collision mesh filename=file:///home/yeshi/icub-gazebo/icub/meshes/collision/icub_s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 scale=1 1 1; visual mesh filename=file:///home/yeshi/icub-gazebo/icub/meshes/visual/icub_l_th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 scale=1 1 1
- link neck_1: geometry collision mesh filename=file:///home/yeshi/icub-gazebo/icub/meshes/collision/icub_s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 scale=1 1 1; visual mesh filename=file:///home/yeshi/icub-gazebo/icub/meshes/visual/icub_neck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 scale=1 1 1
- link neck_2: geometry collision mesh filename=file:///home/yeshi/icub-gazebo/icub/meshes/collision/icub_s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 scale=1 1 1; visual mesh filename=file:///home/yeshi/icub-gazebo/icub/meshes/visual/icub_neck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 scale=1 1 1
- link r_ankle_1: geometry collision mesh filename=file:///home/yeshi/icub-gazebo/icub/meshes/collision/icub_s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 scale=1 1 1; visual mesh filename=file:///home/yeshi/icub-gazebo/icub/meshes/visual/icub_r_an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 scale=1 1 1
- link r_foot: geometry collision mesh filename=file:///home/yeshi/icub-gazebo/icub/meshes/collision/icub_s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 scale=1 1 1; visual mesh filename=file:///home/yeshi/icub-gazebo/icub/meshes/visual/icub_r_fo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 scale=1 1 1
- link r_forearm: geometry collision mesh filename=file:///home/yeshi/icub-gazebo/icub/meshes/collision/icub_s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 scale=1 1 1; visual mesh filename=file:///home/yeshi/icub-gazebo/icub/meshes/visual/icub_r_fo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 scale=1 1 1
- link r_hand: mass 0.213 -> 0.010; geometry collision mesh filename=file:///home/yeshi/icub-gazebo/icub/meshes/collision/r_hand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; collision mesh filename=file:///home/yeshi/icub-gazebo/icub/meshes/collision/r_hand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
- link r_hip_1: geometry collision mesh filename=file:///home/yeshi/icub-gazebo/icub/meshes/collision/icub_s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 scale=1 1 1; visual mesh filename=file:///home/yeshi/icub-gazebo/icub/meshes/visual/icub_r_hi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 scale=1 1 1
- link r_hip_2: geometry collision mesh filename=file:///home/yeshi/icub-gazebo/icub/meshes/collision/icub_s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 scale=1 1 1; visual mesh filename=file:///home/yeshi/icub-gazebo/icub/meshes/visual/icub_r_hi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 scale=1 1 1
- link r_lower_leg: geometry collision mesh filename=file:///home/yeshi/icub-gazebo/icub/meshes/collision/icub_s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 scale=1 1 1; visual mesh filename=file:///home/yeshi/icub-gazebo/icub/meshes/visual/icub_r_sh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 scale=1 1 1
- link r_shoulder_1: geometry collision mesh filename=file:///home/yeshi/icub-gazebo/icub/meshes/collision/icub_s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 scale=1 1 1; visual mesh filename=file:///home/yeshi/icub-gazebo/icub/meshes/visual/icub_r_sh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 scale=1 1 1
- link r_shoulder_2: geometry collision mesh filename=file:///home/yeshi/icub-gazebo/icub/meshes/collision/icub_s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 scale=1 1 1; visual mesh filename=file:///home/yeshi/icub-gazebo/icub/meshes/visual/icub_r_sh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 scale=1 1 1
- link r_upper_arm: geometry collision mesh filename=file:///home/yeshi/icub-gazebo/icub/meshes/collision/icub_s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 scale=1 1 1; visual mesh filename=file:///home/yeshi/icub-gazebo/icub/meshes/visual/icub_r_ar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 scale=1 1 1
- link r_upper_leg: geometry collision mesh filename=file:///home/yeshi/icub-gazebo/icub/meshes/collision/icub_s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 scale=1 1 1; visual mesh filename=file:///home/yeshi/icub-gazebo/icub/meshes/visual/icub_r_th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 scale=1 1 1
- link root_link: geometry collision mesh filename=file:///home/yeshi/icub-gazebo/icub/meshes/collision/icub_s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 scale=1 1 1; visual mesh filename=file:///home/yeshi/icub-gazebo/icub/meshes/visual/icub_root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 scale=1 1 1
- link torso_1: geometry collision mesh filename=file:///home/yeshi/icub-gazebo/icub/meshes/collision/icub_s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 scale=1 1 1; visual mesh filename=file:///home/yeshi/icub-gazebo/icub/meshes/visual/icub_lap_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 scale=1 1 1
Joints:
- removed joint l_gripper_joint
- removed joint r_gripper_joint
- added joint l_aij3: type revolute, parent l_ai_dummy, child l_ail1, origin xyz=0.012 0 0 rpy=1.5708 0 0, axis -0.095753 -0.017412 0.995253, limit lower=0 upper=1.5708 effort=10 velocity=0.5
- added joint l_aij4: type revolute, parent l_ail1, child l_ail2, origin xyz=0.0259 0 0 rpy=0 0 0, axis -0.095753 -0.017412 0.995253, limit lower=0 upper=1.5708 effort=10 velocity=0.5
- added joint l_aij5: type revolute, parent l_ail2, child l_ail3, origin xyz=0.022 0 0 rpy=0 0 0, axis -0.095753 -0.017412 0.995253, limit lower=0 upper=1.5708 effort=10 velocity=0.5
- added joint l_aij6: type revolute, parent l_hand, child l_ai_dummy, origin xyz=0.01225 -0.0643 -0.027 rpy=-1.4749 0.017507 -1.57079, axis -1 0 0, limit lower=-1.5708 upper=1.5708 effort=10 velocity=0.5
- added joint l_lij3: type revolute, parent l_li_dummy, child l_lil1, origin xyz=0.0148 0 0 rpy=1.5708 0 0, axis 0.087189 0.017426 0.996039, limit lower=0 upper=1.5708 effort=10 velocity=0.5
- added joint l_lij4: type revolute, parent l_lil1, child l_lil2, origin xyz=0.0257 0.0 -0.001 rpy=0 0 0, axis 0.087189 0.017426 0.996039, limit lower=0 upper=1.5708 effort=10 velocity=0.5
- added joint l_lij5: type revolute, parent l_lil2, child l_lil3, origin xyz=0.02 0 -0.00385 rpy=0 0 0, axis 0.087189 0.017426 0.996039, limit lower=0 upper=1.5708 effort=10 velocity=0.5
- added joint l_lij6: type revolute, parent l_hand, child l_li_dummy, origin xyz=0.0135 -0.06225 0.02475 rpy=-1.6581 -0.017493 -1.57079, axis -1 0 0, limit lower=-1.5708 upper=1.5708 effort=10 velocity=0.5
- added joint l_mj3: type revolute, parent l_ml_dummy, child l_ml1, origin xyz=0.015 0 0 rpy=1.5708 0 0, axis 0 -7e-06 1, limit lower=0 upper=1.5708 effort=10 velocity=0.5
- added joint l_mj4: type revolute, parent l_ml1, child l_ml2, origin xyz=0.0285 0 0 rpy=0 0 0, axis 0 -7e-06 1, limit lower=0 upper=1.5708 effort=10 velocity=0.5
- added joint l_mj5: type revolute, parent l_ml2, child l_ml3, origin xyz=0.0240 0 0 rpy=0 0 0, axis 0 -7e-06 1, limit lower=0 upper=1.5708 effort=10 velocity=0.5
- added joint l_mj6: type revolute, parent l_hand, child l_ml_dummy, origin xyz=0.011 -0.0653 -0.01 rpy=-1.5708 7e-06 -1.57079, axis -1 0 0, limit lower=-1.5708 upper=1.5708 effort=10 velocity=0.5
- added joint l_rij3: type revolute, parent l_ril_dummy, child l_ril1, origin xyz=0.0148 0 0 rpy=1.5708 0 0, axis 0.087189 0.00866 0.996154, limit lower=0 upper=1.5708 effort=10 velocity=0.5
- added joint l_rij4: type revolute, parent l_ril1, child l_ril2, origin xyz=0.0259 0 0 rpy=0 0 0, axis 0.087189 0.00866 0.996154, limit lower=0 upper=1.5708 effort=10 velocity=0.5
- added joint l_rij5: type revolute, parent l_ril2, child l_ril3, origin xyz=0.0242 0 0.0045 rpy=0 0 0, axis 0.087189 0.00866 0.996154, limit lower=0 upper=1.5708 effort=10 velocity=0.5
- added joint l_rij6: type revolute, parent l_hand, child l_ril_dummy, origin xyz=0.01175 -0.06415 0.0059 rpy=-1.6581 -0.008693 -1.57079, axis 1 0 0, limit lower=-1.5708 upper=1.5708 effort=10 velocity=0.5
- added joint l_tj2: type revolute, parent l_hand, child l_tl0, origin xyz=0.021 -0.0386 -0.01235 rpy=-3.063 1.07329 -1.5708, axis -0.078511 -0.876064 0.47576, limit lower=0 upper=1.5708 effort=10 velocity=0.5
- added joint l_tj4: type revolute, parent l_tl0, child l_tl2, origin xyz=0.021 -0.0056 0 rpy=1.5708 0 0, axis -0.996914 0.068991 -0.037465, limit lower=0 upper=1.5708 effort=10 velocity=0.5
- added joint l_tj5: type revolute, parent l_tl2, child l_tl3, origin xyz=0.026 0 0 rpy=0 0 0, axis -0.996914 0.068991 -0.037465, limit lower=0 upper=1.5708 effort=10 velocity=0.5
- added joint l_tj6: type revolute, parent l_tl3, child l_tl4, origin xyz=0.022 0 0 rpy=0 0 0, axis -0.996914 0.068991 -0.037465, limit lower=0 upper=1.5708 effort=10 velocity=0.5
- added joint r_aij3: type revolute, parent r_ai_dummy, child r_ail1, origin xyz=0.0148 0 0 rpy=1.5708 0 0, axis -0.095753 -0.017426 0.995253, limit lower=0 upper=1.5708 effort=10 velocity=0.5
- added joint r_aij4: type revolute, parent r_ail1, child r_ail2, origin xyz=0.0259 0 0 rpy=0 0 0, axis -0.095753 -0.017426 0.995253, limit lower=0 upper=1.5708 effort=10 velocity=0.5
- added joint r_aij5: type revolute, parent r_ail2, child r_ail3, origin xyz=0.022 0 0 rpy=0 0 0, axis -0.095753 -0.017426 0.995253, limit lower=0 upper=1.5708 effort=10 velocity=0.5
- added joint r_aij6: type revolute, parent r_hand, child r_ai_dummy, origin xyz=0.01225 -0.0643 0.027 rpy=-1.6667 0.017507 -1.57079, axis 1 0 0, limit lower=-1.5708 upper=1.5708 effort=10 velocity=0.5
- added joint r_lij3: type revolute, parent r_li_dummy, child r_lil1, origin xyz=0.0148 0 0 rpy=1.5708 0 0, axis -0.087189 -0.01744 0.996039, limit lower=0 upper=1.5708 effort=10 velocity=0.5
- added joint r_lij4: type revolute, parent r_lil1, child r_lil2, origin xyz=0.0257 0.0 -0.001 rpy=0 0 0, axis -0.087189 -0.01744 0.996039, limit lower=0 upper=1.5708 effort=10 velocity=0.5
- added joint r_lij5: type revolute, parent r_lil2, child r_lil3, origin xyz=0.02 0 -0.00385 rpy=0 0 0, axis -0.087189 -0.01744 0.996039, limit lower=0 upper=1.5708 effort=10 velocity=0.5
- added joint r_lij6: type revolute, parent r_hand, child r_li_dummy, origin xyz=0.0135 -0.06225 -0.02475 rpy=-1.4835 0.017507 -1.57079, axis 1 0 0, limit lower=-1.5708 upper=1.5708 effort=10 velocity=0.5
- added joint r_mj3: type revolute, parent r_m_dummy, child r_ml1, origin xyz=0.015 0 0 rpy=1.5708 0 0, axis 0 -7e-06 1, limit lower=0 upper=1.5708 effort=10 velocity=0.5
- added joint r_mj4: type revolute, parent r_ml1, child r_ml2, origin xyz=0.0285 0 0 rpy=0 0 0, axis 0 -7e-06 1, limit lower=0 upper=1.5708 effort=10 velocity=0.5
- added joint r_mj5: type revolute, parent r_ml2, child r_ml3, origin xyz=0.0240 0 0 rpy=0 0 0, axis 0 -7e-06 1, limit lower=0 upper=1.5708 effort=10 velocity=0.5
- added joint r_mj6: type revolute, parent r_hand, child r_m_dummy, origin xyz=0.011 -0.0653 0.01 rpy=-1.5708 7e-06 -1.57079, axis 1 0 0, limit lower=-1.5708 upper=1.5708 effort=10 velocity=0.5
- added joint r_rij3: type revolute, parent r_rir_dummy, child r_ril1, origin xyz=0.0148 0 0 rpy=1.5708 0 0, axis -0.087189 -0.008674 0.996154, limit lower=0 upper=1.5708 effort=10 velocity=0.5
- added joint r_rij4: type revolute, parent r_ril1, child r_ril2, origin xyz=0.0259 0 0 rpy=0 0 0, axis -0.087189 -0.008674 0.996154, limit lower=0 upper=1.5708 effort=10 velocity=0.5
- added joint r_rij5: type revolute, parent r_ril2, child r_ril3, origin xyz=0.022 0 -0.0045 rpy=0 0 0, axis -0.087189 -0.008674 0.996154, limit lower=0 upper=1.5708 effort=10 velocity=0.5
- added joint r_rij6: type revolute, parent r_hand, child r_rir_dummy, origin xyz=0.01175 -0.06415 -0.0059 rpy=-1.4835 0.008707 -1.57079, axis 1 0 0, limit lower=-1.5708 upper=1.5708 effort=10 velocity=0.5
- added joint r_tj2: type revolute, parent r_hand, child r_tl0, origin xyz=0.021 -0.0386 0.01235 rpy=-0.078604 -1.07329 -1.57079, axis 0.078514 0.876064 0.47576, limit lower=0 upper=1.5708 effort=10 velocity=0.5
- added joint r_tj4: type revolute, parent r_tl0, child r_tl2, origin xyz=0.021 0.0056 0 rpy=-1.5708 0 0, axis 0.996913 -0.068997 -0.037476, limit lower=0 upper=1.5708 effort=10 velocity=0.5
- added joint r_tj5: type revolute, parent r_tl2, child r_tl3, origin xyz=0.026 0 0 rpy=0 0 0, axis 0.996913 -0.068997 -0.037476, limit lower=0 upper=1.5708 effort=10 velocity=0.5
- added joint r_tj6: type revolute, parent r_tl3, child r_tl4, origin xyz=0.022 0 0 rpy=0 0 0, axis 0.996913 -0.068997 -0.037476, limit lower=0 upper=1.5708 effort=10 velocity=0.5
- joint l_hand_dh_frame_fixed_joint: origin xyz=0.0625 0 -0.016 rpy=0 -0 0 -> xyz=0.025 -0.04 0 rpy=0 -0 0
- joint r_hand_dh_frame_fixed_joint: origin xyz=0.0625 0 0.016 rpy=0 -0 0 -> xyz=0.025 -0.04 0 rpy=0 -0 0
